File: 2-Hardware/SingleEncoder/SingleEncoder.sch (KiCad schematic (older format))
At the start: 25 parts, among them J1 PMOD_SINGLE, P1 CONN_01X06, Q1 MMBT2222, Q2 MMBT2222, U1 TPS60131, U2 MCP6L02, U3 ILD213T

Commit message: Started footprint association
Parts:
- C1, C2, C3, C4, C5, R1, R2, R3, R4, R5, R6, R7, R8, R9: footprint (none) -> SMD:SMD_0805
- D1: footprint (none) -> LEDs:LED_1206
- J1: footprint (none) -> Connectors:PMOD_SINGLE_MALE
- TP1, TP2, TP3: footprint (none) -> Connectors:TESTPOINT_063

Commit message: Associated DIN footprint
Parts:
- P1: footprint (none) -> Connectors:DIN_CUI_SDS-50J
Changed lines of the file:
@@
 F 0 "P1" H 1600 4800 50  0000 C CNN
 F 1 "CONN_01X06" V 1700 4450 50  0000 C CNN
-F 2 "" H 1600 4450 60  0001 C CNN
+F 2 "Connectors:DIN_CUI_SDS-50J" H 1600 4450 60  0001 C CNN
 F 3 "" H 1600 4450 60  0000 C CNN
 	1    1600 4450

Commit message: Finished footprint association
Parts:
- Q1, Q2: footprint (none) -> Transistors:TRANS_SOT-23-3_BEC
- U1: footprint (none) -> SMD:SSOP_20_4.5mm_6.6mm_0.65mm_PWP
- U2: footprint (none) -> SMD:SSOP_08_3.0mm_3.0mm_0.65mm
- U3: footprint (none) -> SMD:SOIC_08_4.0mm_5.8mm_1.27mm
Changed lines of the file:
@@
 F 0 "U1" H 4300 1400 60  0000 C CNN
 F 1 "TPS60131" H 3700 1950 60  0000 C CNN
-F 2 "" H 3300 1700 60  0001 C CNN
+F 2 "SMD:SSOP_20_4.5mm_6.6mm_0.65mm_PWP" H 3300 1700 60  0001 C CNN
 F 3 "http://www.ti.com/lit/ds/symlink/tps60130.pdf" H 3300 1700 60  0001 C CNN
 F 4 "296-2272-5-ND" H 3700 1950 60  0001 C CNN "DigikeyNumber"
@@
 F 0 "U2" H 7900 2150 60  0000 C CNN
 F 1 "MCP6L02" H 7950 1600 60  0000 C CNN
-F 2 "" H 7900 3150 60  0001 C CNN
+F 2 "SMD:SSOP_08_3.0mm_3.0mm_0.65mm" H 7900 3150 60  0001 C CNN
 F 3 "http://ww1.microchip.com/downloads/en/DeviceDoc/22140b.pdf" H 8000 2750 60  0001 C CNN
 F 4 "MCP6L02T-E/MSCT-ND" H 8000 2900 60  0001 C CNN "DigikeyNumber"
@@
 F 0 "U2" H 7900 3850 60  0000 C CNN
 F 1 "MCP6L02" H 7950 3300 60  0000 C CNN
-F 2 "" H 7900 4850 60  0001 C CNN
+F 2 "SMD:SSOP_08_3.0mm_3.0mm_0.65mm" H 7900 4850 60  0001 C CNN
 F 3 "http://ww1.microchip.com/downloads/en/DeviceDoc/22140b.pdf" H 8000 4450 60  0001 C CNN
 F 4 "MCP6L02T-E/MSCT-ND" H 8000 4600 60  0001 C CNN "DigikeyNumber"
@@
 F 0 "U3" H 9500 2200 60  0000 C CNN
 F 1 "ILD213T" H 9300 1700 60  0000 C CNN
-F 2 "" H 9300 1950 60  0001 C CNN
+F 2 "SMD:SOIC_08_4.0mm_5.8mm_1.27mm" H 9300 1950 60  0001 C CNN
 F 3 "http://www.vishay.com/docs/83647/ild205t.pdf" H 9400 2300 60  0001 C CNN
 F 4 "751-1312-1-ND" H 9750 2400 60  0001 C CNN "DigikeyNumber"
@@
 F 0 "U3" H 9500 3900 60  0000 C CNN
 F 1 "ILD213T" H 9300 3400 60  0000 C CNN
-F 2 "" H 9300 3650 60  0001 C CNN
+F 2 "SMD:SOIC_08_4.0mm_5.8mm_1.27mm" H 9300 3650 60  0001 C CNN
 F 3 "http://www.vishay.com/docs/83647/ild205t.pdf" H 9400 4000 60  0001 C CNN
 F 4 "751-1312-1-ND" H 9750 4100 60  0001 C CNN "DigikeyNumber"
@@
 F 0 "Q2" H 10310 3720 60  0000 R CNN
 F 1 "MMBT2222" H 10310 3400 60  0000 R CNN
-F 2 "" H 10210 3620 60  0001 C CNN
+F 2 "Transistors:TRANS_SOT-23-3_BEC" H 10210 3620 60  0001 C CNN
 F 3 "https://www.fairchildsemi.com/datasheets/MM/MMBT2222.pdf" H 10310 3720 60  0001 C CNN
 F 4 "MMBT2222AFSCT-ND" H 10300 3550 60  0001 C CNN "DigikeyNumber"
@@
 F 0 "Q1" H 10310 2020 60  0000 R CNN
 F 1 "MMBT2222" H 10310 1700 60  0000 R CNN
-F 2 "" H 10210 1920 60  0001 C CNN
+F 2 "Transistors:TRANS_SOT-23-3_BEC" H 10210 1920 60  0001 C CNN
 F 3 "https://www.fairchildsemi.com/datasheets/MM/MMBT2222.pdf" H 10310 2020 60  0001 C CNN
 F 4 "MMBT2222AFSCT-ND" H 10300 1850 60  0001 C CNN "DigikeyNumber"

Commit message: Started circuit board layout
Parts:
- removed R2: 0, SMD:SMD_0805, symbol RES
- added C2: 15uF, SMD:SMD_0805, symbol CAP
- added C5: 33uF, SMD:SMD_0805, symbol CAP
- renumbered C2 to C3, C3 to C4, C4 to C6, C5 to C7, R9 to R2
Connections:
- net +5V: now also C5.1
- net GND: now also J1.5 (GND), U1.1 (GND), U1.19 (GND), U1.2 (GND), U1.20 (GND), U3.2 (IN_C), U3.4 (IN_C), U3.5 (OUT_E), U3.7 (OUT_E), C2.2, C5.2; no longer J1.6 (VCC), U3.2 (IN_C), U3.4 (IN_C), U3.5 (OUT_E), U3.7 (OUT_E)
- net LOGIC_A: now also J1.1 (IO_1); no longer J1.4 (IO_4)
- net LOGIC_B: now also J1.2 (IO_2); no longer J1.3 (IO_3)
- net PWR_EN: now also J1.3 (IO_3); no longer J1.2 (IO_2)
- net VCC: now also J1.6 (VCC), C2.1; no longer J1.5 (GND)
- net at R3.1: now also U3.1 (IN_A); no longer U3.1 (IN_A)
- net at Q1.B, R5.2: now also U3.8 (OUT_C); no longer U3.8 (OUT_C)
- net at R4.1: now also U3.3 (IN_A); no longer U3.3 (IN_A)
- net at Q2.B, R6.2: now also U3.6 (OUT_C); no longer U3.6 (OUT_C)
Other:
- moved on the sheet: C6
Changed lines of the file:
@@
 F 3 "" H 1250 2000 60  0000 C CNN
 	1    1100 2000
-	1    0    0    1
+	1    0    0    -1
 $EndComp
 $Comp
@@
 $EndComp
 $Comp
-L CAP C2
+L CAP C3
 U 1 1 55A55E3A
 P 2800 2150
-F 0 "C2" H 2800 2220 60  0000 R CNN
+F 0 "C3" H 2800 2220 60  0000 R CNN
 F 1 "2.2uF" H 2800 2070 60  0000 R CNN
 F 2 "SMD:SMD_0805" V 2540 2050 60  0001 C CNN
@@
 $EndComp
 $Comp
-L CAP C3
+L CAP C4
 U 1 1 55A55E5F
 P 4700 2150
-F 0 "C3" H 4700 2220 60  0000 R CNN
+F 0 "C4" H 4700 2220 60  0000 R CNN
 F 1 "2.2uF" H 4700 2070 60  0000 R CNN
 F 2 "SMD:SMD_0805" V 4440 2050 60  0001 C CNN
@@
 $EndComp
 $Comp
-L CAP C4
+L CAP C6
 U 1 1 55A563BE
-P 5150 1850
-F 0 "C4" H 5150 1920 60  0000 R CNN
-F 1 "33uF" H 5150 1770 60  0000 R CNN
-F 2 "SMD:SMD_0805" V 4890 1750 60  0001 C CNN
-F 3 "" V 4990 1850 60  0001 C CNN
-	1    5150 1850
+P 5200 1850
+F 0 "C6" H 5200 1920 60  0000 R CNN
+F 1 "33uF" H 5200 1770 60  0000 R CNN
+F 2 "SMD:SMD_0805" V 4940 1750 60  0001 C CNN
+F 3 "" V 5040 1850 60  0001 C CNN
+	1    5200 1850
 	1    0    0    -1
 $EndComp
@@
 L GND #PWR05
 U 1 1 55A563F5
-P 5150 2100
-F 0 "#PWR05" H 5150 1850 50  0001 C CNN
-F 1 "GND" H 5150 1950 50  0000 C CNN
-F 2 "" H 5150 2100 60  0000 C CNN
-F 3 "" H 5150 2100 60  0000 C CNN
-	1    5150 2100
-	1    0    0    -1
-$EndComp
-Wire Wire Line
-	5150 2100 5150 2050
-Wire Wire Line
-	5150 1550 5150 1650
+P 5200 2150
+F 0 "#PWR05" H 5200 1900 50  0001 C CNN
+F 1 "GND" H 5200 2000 50  0000 C CNN
+F 2 "" H 5200 2150 60  0000 C CNN
+F 3 "" H 5200 2150 60  0000 C CNN
+	1    5200 2150
+	1    0    0    -1
+$EndComp
+Wire Wire Line
+	5200 2050 5200 2150
+Wire Wire Line
+	5200 1550 5200 1650
 Wire Wire Line
 	4500 1550 5500 1550
@@
 	4600 1650 4500 1650
 Connection ~ 4600 1550
-Connection ~ 5150 1550
 $Comp
 L +5V #PWR06
@@
 L GND #PWR07
 U 1 1 55A56863
-P 2450 2050
-F 0 "#PWR07" H 2450 1800 50  0001 C CNN
-F 1 "GND" H 2450 1900 50  0000 C CNN
-F 2 "" H 2450 2050 60  0000 C CNN
-F 3 "" H 2450 2050 60  0000 C CNN
-	1    2450 2050
+P 2450 2100
+F 0 "#PWR07" H 2450 1850 50  0001 C CNN
+F 1 "GND" H 2450 1950 50  0000 C CNN
+F 2 "" H 2450 2100 60  0000 C CNN
+F 3 "" H 2450 2100 60  0000 C CNN
+	1    2450 2100
 	1    0    0    -1
 $EndComp
@@
 Connection ~ 2650 1550
 Wire Wire Line
-	2450 2000 2450 2050
+	2450 2000 2450 2100
 $Comp
 L GND #PWR08
 U 1 1 55A56ABE
-P 3450 2900
-F 0 "#PWR08" H 3450 2650 50  0001 C CNN
-F 1 "GND" H 3450 2750 50  0000 C CNN
-F 2 "" H 3450 2900 60  0000 C CNN
-F 3 "" H 3450 2900 60  0000 C CNN
-	1    3450 2900
-	1    0    0    -1
-$EndComp
-$Comp
-L RES R2
-U 1 1 55A56AE0
 P 3700 2800
-F 0 "R2" V 3800 2800 60  0000 C CNN
-F 1 "0" V 3700 2800 60  0000 C CNN
-F 2 "SMD:SMD_0805" V 3440 2700 60  0001 C CNN
-F 3 "" V 3540 2800 60  0001 C CNN
+F 0 "#PWR08" H 3700 2550 50  0001 C CNN
+F 1 "GND" H 3700 2650 50  0000 C CNN
+F 2 "" H 3700 2800 60  0000 C CNN
+F 3 "" H 3700 2800 60  0000 C CNN
 	1    3700 2800
-	0    1    1    0
+	1    0    0    -1
 $EndComp
 Wire Wire Line
@@
 Wire Wire Line
 	4050 2650 4050 2550
-Wire Wire Line
-	3950 2550 3950 2800
 Connection ~ 3950 2650
 Wire Wire Line
-	3850 2550 3850 2650
+	3850 2750 3850 2550
 Connection ~ 3850 2650
 Wire Wire Line
-	3950 2800 3900 2800
-Wire Wire Line
 	3650 2650 3650 2550
 Wire Wire Line
@@
 Wire Wire Line
 	3350 2650 3350 2550
-Wire Wire Line
-	3450 2550 3450 2900
 Connection ~ 3450 2650
 Wire Wire Line
-	3550 2550 3550 2650
+	3550 2550 3550 2750
 Connection ~ 3550 2650
-Wire Wire Line
-	3450 2800 3500 2800
-Connection ~ 3450 2800
 Text Notes 650  750  0    100  ~ 0
 PMOD Connector
@@
 	7650 2250 7650 2200
 $Comp
-L CAP C5
+L CAP C7
 U 1 1 55A58249
 P 8100 1450
-F 0 "C5" H 8100 1520 60  0000 R CNN
+F 0 "C7" H 8100 1520 60  0000 R CNN
 F 1 "0.1uF" H 8100 1370 60  0000 R CNN
 F 2 "SMD:SMD_0805" V 7840 1350 60  0001 C CNN
@@
 $Comp
 L ILD213T U3
-U 1 1 55A592A9
+U 2 1 55A592A9
+P 9300 3650
+F 0 "U3" H 9500 3900 60  0000 C CNN
+F 1 "ILD213T" H 9300 3400 60  0000 C CNN
+F 2 "SMD:SOIC_08_4.0mm_5.8mm_1.27mm" H 9300 3650 60  0001 C CNN
+F 3 "http://www.vishay.com/docs/83647/ild205t.pdf" H 9400 4000 60  0001 C CNN
+F 4 "751-1312-1-ND" H 9750 4100 60  0001 C CNN "DigikeyNumber"
+F 5 "Vishay" H 9750 4250 60  0001 C CNN "Manufacturer"
+F 6 "ILD213T" H 9800 4350 60  0001 C CNN "ManufacturerNumber"
+	2    9300 3650
+	1    0    0    -1
+$EndComp
+$Comp
+L ILD213T U3
+U 1 1 55A59311
 P 9300 1950
 F 0 "U3" H 9500 2200 60  0000 C CNN
@@
 $EndComp
 $Comp
-L ILD213T U3
-U 2 1 55A59311
-P 9300 3650
-F 0 "U3" H 9500 3900 60  0000 C CNN
-F 1 "ILD213T" H 9300 3400 60  0000 C CNN
-F 2 "SMD:SOIC_08_4.0mm_5.8mm_1.27mm" H 9300 3650 60  0001 C CNN
-F 3 "http://www.vishay.com/docs/83647/ild205t.pdf" H 9400 4000 60  0001 C CNN
-F 4 "751-1312-1-ND" H 9750 4100 60  0001 C CNN "DigikeyNumber"
-F 5 "Vishay" H 9750 4250 60  0001 C CNN "Manufacturer"
-F 6 "ILD213T" H 9800 4350 60  0001 C CNN "ManufacturerNumber"
-	2    9300 3650
-	1    0    0    -1
-$EndComp
-$Comp
 L GND #PWR015
 U 1 1 55A593CB
@@
 LOGIC_A
 Wire Wire Line
-	10800 1600 10400 1600
+	10400 1600 10800 1600
 Connection ~ 10400 1600
 $Comp
@@
 	2100 5100 500  5100
 $Comp
-L RES R9
+L RES R2
 U 1 1 55A5D293
 P 5500 1800
-F 0 "R9" V 5600 1800 60  0000 C CNN
+F 0 "R2" V 5600 1800 60  0000 C CNN
 F 1 "330" V 5500 1800 60  0000 C CNN
 F 2 "SMD:SMD_0805" V 5240 1700 60  0001 C CNN
@@
 Wire Wire Line
 	10700 3950 10700 4050
+$Comp
+L CAP C2
+U 1 1 55A82F72
+P 2700 1800
+F 0 "C2" H 2700 1870 60  0000 R CNN
+F 1 "15uF" H 2700 1720 60  0000 R CNN
+F 2 "SMD:SMD_0805" V 2440 1700 60  0001 C CNN
+F 3 "" V 2540 1800 60  0001 C CNN
+	1    2700 1800
+	1    0    0    -1
+$EndComp
+Wire Wire Line
+	2700 2000 2700 2050
+Wire Wire Line
+	2700 2050 2450 2050
+Connection ~ 2450 2050
+Wire Wire Line
+	2700 1600 2700 1550
+Connection ~ 2700 1550
+$Comp
+L CAP C5
+U 1 1 55A83372
+P 4950 1850
+F 0 "C5" H 4950 1920 60  0000 R CNN
+F 1 "33uF" H 4950 1770 60  0000 R CNN
+F 2 "SMD:SMD_0805" V 4690 1750 60  0001 C CNN
+F 3 "" V 4790 1850 60  0001 C CNN
+	1    4950 1850
+	1    0    0    -1
+$EndComp
+Wire Wire Line
+	4950 1650 4950 1550
+Wire Wire Line
+	4950 2050 4950 2100
+Wire Wire Line
+	4950 2100 5200 2100
+Connection ~ 5200 2100
+Connection ~ 5200 1550
+Connection ~ 4950 1550
+Wire Wire Line
+	3450 2550 3450 2650
+Wire Wire Line
+	3950 2550 3950 2650
+Wire Wire Line
+	3700 2750 3700 2800
+Connection ~ 3700 2750
+Wire Wire Line
+	3550 2750 3850 2750
 $EndSCHEMATC

Commit message: Finalized BOM
Parts:
- C1, C2: DigikeyNumber (none) -> 445-14362-1-ND; Manufacturer (none) -> TDK Corporation; ManufacturerNumber (none) -> C2012X5R1A156M085AC
- C3, C4: DigikeyNumber (none) -> 445-1588-1-ND; Manufacturer (none) -> TDK Corporation; ManufacturerNumber (none) -> C2012X5R1A225K085AA
- C5, C6: DigikeyNumber (none) -> 445-8238-1-ND; Manufacturer (none) -> TDK Corporation; ManufacturerNumber (none) -> C2012X5R1A336M125AC
- C7: DigikeyNumber (none) -> 311-1141-1-ND; Manufacturer (none) -> Yageo; ManufacturerNumber (none) -> CC0805KRX7R8BB104
- D1: DigikeyNumber (none) -> 754-1137-1-ND; Manufacturer (none) -> Kingbright; ManufacturerNumber (none) -> APT3216EC
- J1: DigikeyNumber (none) -> 609-3313-ND; Manufacturer (none) -> FCI; ManufacturerNumber (none) -> 68016-106HLF
- P1: DigikeyNumber (none) -> CP-2350-ND; Manufacturer (none) -> CUI Inc; ManufacturerNumber (none) -> SDS-50J
- R1, R5, R6, R7, R8: DigikeyNumber (none) -> P10.0KCCT-ND; Manufacturer (none) -> Panasonic Electronic Components; ManufacturerNumber (none) -> ERJ-6ENF1002V
- R2: DigikeyNumber (none) -> P330CCT-ND; Manufacturer (none) -> Panasonic Electronic Components; ManufacturerNumber (none) -> ERJ-6ENF3300V
- R3, R4: DigikeyNumber (none) -> P220CCT-ND; Manufacturer (none) -> Panasonic Electronic Components; ManufacturerNumber (none) -> ERJ-6ENF2200V
Connections:
- net at U3.3 (IN_A): now also R3.1; no longer R4.1
- net at Q2.B, R6.2: now also U3.8 (OUT_C); no longer U3.6 (OUT_C)
- net at U3.1 (IN_A): now also R4.1; no longer R3.1
- net at Q1.B, R5.2: now also U3.6 (OUT_C); no longer U3.8 (OUT_C)
Other:
- moved on the sheet: U3A, U3B
Changed lines of the file:
@@
 F 2 "Connectors:PMOD_SINGLE_MALE" H 1250 2000 60  0001 C CNN
 F 3 "" H 1250 2000 60  0000 C CNN
+F 4 "609-3313-ND" H 1100 2000 60  0001 C CNN "DigikeyNumber"
+F 5 "FCI" H 1100 2000 60  0001 C CNN "Manufacturer"
+F 6 "68016-106HLF" H 1100 2000 60  0001 C CNN "ManufacturerNumber"
 	1    1100 2000
 	1    0    0    -1
@@
 F 2 "SMD:SMD_0805" V 3090 850 60  0001 C CNN
 F 3 "" V 3190 950 60  0001 C CNN
+F 4 "P10.0KCCT-ND" H 3350 950 60  0001 C CNN "DigikeyNumber"
+F 5 "Panasonic Electronic Components" H 3350 950 60  0001 C CNN "Manufacturer"
+F 6 "ERJ-6ENF1002V" H 3350 950 60  0001 C CNN "ManufacturerNumber"
 	1    3350 950
 	1    0    0    -1
@@
 F 2 "SMD:SMD_0805" V 2540 2050 60  0001 C CNN
 F 3 "" V 2640 2150 60  0001 C CNN
+F 4 "445-1588-1-ND" H 2800 2150 60  0001 C CNN "DigikeyNumber"
+F 5 "TDK Corporation" H 2800 2150 60  0001 C CNN "Manufacturer"
+F 6 "C2012X5R1A225K085AA" H 2800 2150 60  0001 C CNN "ManufacturerNumber"
 	1    2800 2150
 	1    0    0    -1
@@
 F 2 "SMD:SMD_0805" V 4440 2050 60  0001 C CNN
 F 3 "" V 4540 2150 60  0001 C CNN
+F 4 "445-1588-1-ND" H 4700 2150 60  0001 C CNN "DigikeyNumber"
+F 5 "TDK Corporation" H 4700 2150 60  0001 C CNN "Manufacturer"
+F 6 "C2012X5R1A225K085AA" H 4700 2150 60  0001 C CNN "ManufacturerNumber"
 	1    4700 2150
 	1    0    0    -1
@@
 F 2 "SMD:SMD_0805" V 4940 1750 60  0001 C CNN
 F 3 "" V 5040 1850 60  0001 C CNN
+F 4 "445-8238-1-ND" H 5200 1850 60  0001 C CNN "DigikeyNumber"
+F 5 "TDK Corporation" H 5200 1850 60  0001 C CNN "Manufacturer"
+F 6 "C2012X5R1A336M125AC" H 5200 1850 60  0001 C CNN "ManufacturerNumber"
 	1    5200 1850
 	1    0    0    -1
@@
 F 2 "SMD:SMD_0805" V 2190 1700 60  0001 C CNN
 F 3 "" V 2290 1800 60  0001 C CNN
+F 4 "445-14362-1-ND" H 2450 1800 60  0001 C CNN "DigikeyNumber"
+F 5 "TDK Corporation" H 2450 1800 60  0001 C CNN "Manufacturer"
+F 6 "C2012X5R1A156M085AC" H 2450 1800 60  0001 C CNN "ManufacturerNumber"
 	1    2450 1800
 	1    0    0    -1
@@
 F 2 "Connectors:DIN_CUI_SDS-50J" H 1600 4450 60  0001 C CNN
 F 3 "" H 1600 4450 60  0000 C CNN
+F 4 "CP-2350-ND" H 1600 4450 60  0001 C CNN "DigikeyNumber"
+F 5 "CUI Inc" H 1600 4450 60  0001 C CNN "Manufacturer"
+F 6 "SDS-50J" H 1600 4450 60  0001 C CNN "ManufacturerNumber"
 	1    1600 4450
 	1    0    0    -1
@@
 F 2 "SMD:SMD_0805" V 7840 1350 60  0001 C CNN
 F 3 "" V 7940 1450 60  0001 C CNN
+F 4 "311-1141-1-ND" H 8100 1450 60  0001 C CNN "DigikeyNumber"
+F 5 "Yageo" H 8100 1450 60  0001 C CNN "Manufacturer"
+F 6 "CC0805KRX7R8BB104" H 8100 1450 60  0001 C CNN "ManufacturerNumber"
 	1    8100 1450
 	0    1    1    0
@@
 L ILD213T U3
 U 2 1 55A592A9
+P 9300 1950
+F 0 "U3" H 9500 2200 60  0000 C CNN
+F 1 "ILD213T" H 9300 1700 60  0000 C CNN
+F 2 "SMD:SOIC_08_4.0mm_5.8mm_1.27mm" H 9300 1950 60  0001 C CNN
+F 3 "http://www.vishay.com/docs/83647/ild205t.pdf" H 9400 2300 60  0001 C CNN
+F 4 "751-1312-1-ND" H 9750 2400 60  0001 C CNN "DigikeyNumber"
+F 5 "Vishay" H 9750 2550 60  0001 C CNN "Manufacturer"
+F 6 "ILD213T" H 9800 2650 60  0001 C CNN "ManufacturerNumber"
+	2    9300 1950
+	1    0    0    -1
+$EndComp
+$Comp
+L ILD213T U3
+U 1 1 55A59311
 P 9300 3650
 F 0 "U3" H 9500 3900 60  0000 C CNN
@@
 F 5 "Vishay" H 9750 4250 60  0001 C CNN "Manufacturer"
 F 6 "ILD213T" H 9800 4350 60  0001 C CNN "ManufacturerNumber"
-	2    9300 3650
-	1    0    0    -1
-$EndComp
-$Comp
-L ILD213T U3
-U 1 1 55A59311
-P 9300 1950
-F 0 "U3" H 9500 2200 60  0000 C CNN
-F 1 "ILD213T" H 9300 1700 60  0000 C CNN
-F 2 "SMD:SOIC_08_4.0mm_5.8mm_1.27mm" H 9300 1950 60  0001 C CNN
-F 3 "http://www.vishay.com/docs/83647/ild205t.pdf" H 9400 2300 60  0001 C CNN
-F 4 "751-1312-1-ND" H 9750 2400 60  0001 C CNN "DigikeyNumber"
-F 5 "Vishay" H 9750 2550 60  0001 C CNN "Manufacturer"
-F 6 "ILD213T" H 9800 2650 60  0001 C CNN "ManufacturerNumber"
-	1    9300 1950
+	1    9300 3650
 	1    0    0    -1
 $EndComp
@@
 F 2 "SMD:SMD_0805" V 8390 1750 60  0001 C CNN
 F 3 "" V 8490 1850 60  0001 C CNN
+F 4 "P220CCT-ND" H 8650 1850 60  0001 C CNN "DigikeyNumber"
+F 5 "Panasonic Electronic Components" H 8650 1850 60  0001 C CNN "Manufacturer"
+F 6 "ERJ-6ENF2200V" H 8650 1850 60  0001 C CNN "ManufacturerNumber"
 	1    8650 1850
 	0    1    1    0
@@
 F 2 "SMD:SMD_0805" V 8390 3450 60  0001 C CNN
 F 3 "" V 8490 3550 60  0001 C CNN
+F 4 "P220CCT-ND" H 8650 3550 60  0001 C CNN "DigikeyNumber"
+F 5 "Panasonic Electronic Components" H 8650 3550 60  0001 C CNN "Manufacturer"
+F 6 "ERJ-6ENF2200V" H 8650 3550 60  0001 C CNN "ManufacturerNumber"
 	1    8650 3550
 	0    1    1    0
@@
 F 2 "SMD:SMD_0805" V 9640 3200 60  0001 C CNN
 F 3 "" V 9740 3300 60  0001 C CNN
+F 4 "P10.0KCCT-ND" H 9900 3300 60  0001 C CNN "DigikeyNumber"
+F 5 "Panasonic Electronic Components" H 9900 3300 60  0001 C CNN "Manufacturer"
+F 6 "ERJ-6ENF1002V" H 9900 3300 60  0001 C CNN "ManufacturerNumber"
 	1    9900 3300
 	1    0    0    -1
@@
 F 2 "SMD:SMD_0805" V 9640 1500 60  0001 C CNN
 F 3 "" V 9740 1600 60  0001 C CNN
+F 4 "P10.0KCCT-ND" H 9900 1600 60  0001 C CNN "DigikeyNumber"
+F 5 "Panasonic Electronic Components" H 9900 1600 60  0001 C CNN "Manufacturer"
+F 6 "ERJ-6ENF1002V" H 9900 1600 60  0001 C CNN "ManufacturerNumber"
 	1    9900 1600
 	1    0    0    -1
@@
 F 2 "SMD:SMD_0805" V 10140 2950 60  0001 C CNN
 F 3 "" V 10240 3050 60  0001 C CNN
+F 4 "P10.0KCCT-ND" H 10400 3050 60  0001 C CNN "DigikeyNumber"
+F 5 "Panasonic Electronic Components" H 10400 3050 60  0001 C CNN "Manufacturer"
+F 6 "ERJ-6ENF1002V" H 10400 3050 60  0001 C CNN "ManufacturerNumber"
 	1    10400 3050
 	1    0    0    -1
@@
 F 2 "SMD:SMD_0805" V 10140 1250 60  0001 C CNN
 F 3 "" V 10240 1350 60  0001 C CNN
+F 4 "P10.0KCCT-ND" H 10400 1350 60  0001 C CNN "DigikeyNumber"
+F 5 "Panasonic Electronic Components" H 10400 1350 60  0001 C CNN "Manufacturer"
+F 6 "ERJ-6ENF1002V" H 10400 1350 60  0001 C CNN "ManufacturerNumber"
 	1    10400 1350
 	1    0    0    -1
@@
 F 2 "SMD:SMD_0805" V 5240 1700 60  0001 C CNN
 F 3 "" V 5340 1800 60  0001 C CNN
+F 4 "P330CCT-ND" H 5500 1800 60  0001 C CNN "DigikeyNumber"
+F 5 "Panasonic Electronic Components" H 5500 1800 60  0001 C CNN "Manufacturer"
+F 6 "ERJ-6ENF3300V" H 5500 1800 60  0001 C CNN "ManufacturerNumber"
 	1    5500 1800
 	1    0    0    -1
@@
 F 2 "LEDs:LED_1206" H 5500 2280 60  0001 C CNN
 F 3 "" H 5500 2280 60  0001 C CNN
+F 4 "754-1137-1-ND" H 5500 2300 60  0001 C CNN "DigikeyNumber"
+F 5 "Kingbright" H 5500 2300 60  0001 C CNN "Manufacturer"
+F 6 "APT3216EC" H 5500 2300 60  0001 C CNN "ManufacturerNumber"
 	1    5500 2300
 	-1   0    0    1
@@
 F 2 "SMD:SMD_0805" V 2440 1700 60  0001 C CNN
 F 3 "" V 2540 1800 60  0001 C CNN
+F 4 "445-14362-1-ND" H 2700 1800 60  0001 C CNN "DigikeyNumber"
+F 5 "TDK Corporation" H 2700 1800 60  0001 C CNN "Manufacturer"
+F 6 "C2012X5R1A156M085AC" H 2700 1800 60  0001 C CNN "ManufacturerNumber"
 	1    2700 1800
 	1    0    0    -1
@@
 F 2 "SMD:SMD_0805" V 4690 1750 60  0001 C CNN
 F 3 "" V 4790 1850 60  0001 C CNN
+F 4 "445-8238-1-ND" H 4950 1850 60  0001 C CNN "DigikeyNumber"
+F 5 "TDK Corporation" H 4950 1850 60  0001 C CNN "Manufacturer"
+F 6 "C2012X5R1A336M125AC" H 4950 1850 60  0001 C CNN "ManufacturerNumber"
 	1    4950 1850
 	1    0    0    -1
